Commit message: gazebo

File: description/robot_core.xacro (robot description, xacro)
@@ -44,4 +44,7 @@
         </xacro:inertial_box>
     </link>
+    <gazebo reference="chassis">
+        <material>Gazebo/White</material>
+    </gazebo>
     <!--LEFT WHEEL LINK-->
     <joint name="left_wheel_joint" type="continuous">
@@ -67,4 +70,7 @@
         </xacro:inertial_cylinder>
     </link>
+    <gazebo reference="left_wheel">
+        <material>Gazebo/Blue</material>
+    </gazebo>
         <!--RIGHT WHEEL LINK-->
     <joint name="right_wheel_joint" type="continuous">
@@ -90,4 +96,7 @@
         </xacro:inertial_cylinder>
     </link>
+        <gazebo reference="right_wheel">
+        <material>Gazebo/Blue</material>
+    </gazebo>
         <!-- CASTER WHEEL LINK -->
     <joint name="caster_wheel_joint" type="fixed">
@@ -105,10 +114,15 @@
         <collision>
             <geometry>
-                <sphere radius="0.05}"/>
+                <sphere radius="0.05"/>
             </geometry>
         </collision>
-    </link>
      <xacro:inertial_sphere mass="0.1" radius="0.05">
             <origin xyz="0 0 0" rpy="0 0 0"/>
-        </xacro:inertial_sphere>
+    </xacro:inertial_sphere>
+   </link>
+           <gazebo reference="caster_wheel">
+        <material>Gazebo/Black</material>
+        <mu1 value ="0.001"/>
+        <mu2 value="0.001"/>
+    </gazebo>
 </robot>
